File: CAD/kiCAD/arduino/arduino.kicad_pcb (KiCad board)
At the start: 2 copper layers, 9 parts

Commit message: Big Updates
Parts:
- removed C1: 10uF, Capacitor_THT:C_Disc_D4.7mm_W2.5mm_P5.00mm
- moved powerIN2 75.1 mm to (159.1, 117.6), turned to 180 degrees
- moved 5Vin1 66.6 mm to (133.9, 117.6), turned to 180 degrees
- moved 5Vbar1 15.2 mm to (138.5, 118.0), turned to 0 degrees
- moved 3.3Vbar1 8.02 mm to (152.5, 118.0), turned to 0 degrees
- moved GNDBar1 5.39 mm to (145.5, 118.0), turned to 0 degrees
- moved Expansion2 3.92 mm to (133.9, 73.7)
- moved Expansion1 3.14 mm to (159.4, 109.3)
- renumbered powerIN1 to 5Vin1
Routing:
- net GND: track 0.08 -> 97.8 mm
- net +5V: track 0.08 -> 51.0 mm
- net +3.3V: track 0.00 -> 37.2 mm
- net RST: track 0.08 -> 25.3 mm
- net nano5V: track 0.08 -> 5.19 mm
- net D13: track 0.08 -> 5.19 mm
- net AREF: track 0.08 -> 5.19 mm
- net A7: track 0.08 -> 5.19 mm
- net A6: track 0.08 -> 5.19 mm
- net A4: track 0.08 -> 5.19 mm
- net A1: track 0.08 -> 5.19 mm
- net nano3.3V: track 0.08 -> 5.11 mm
- net A5: track 0.08 -> 5.11 mm
- net A3: track 0.08 -> 5.11 mm
- net A2: track 0.08 -> 5.11 mm
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Other:
- board outline added: 33.9 x 65.8 mm
- board text added: "+"
- board text added: "+3.3V"
- board text added: "+5V"
- board text added: "-"
- board text added: "3.3Vin"
- board text added: "5Vin"
- board text added: "GND"

Commit message: updates
Parts:
- moved powerIN2 0.28 mm to (159.4, 117.6)
Other:
- board size 33.9 x 65.8 mm -> 35 x 65 mm
Changed lines of the file:
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@@
 		)
 		(property "Value" "Conn_02x05_Counter_Clockwise"
-			(at 1.27 12.49 360)
+			(at 1.27 12.49 0)
 			(layer "F.Fab")
 			(hide yes)
@@
 		)
 		(property "Value" "Conn_02x05_Counter_Clockwise"
-			(at 1.27 12.49 360)
+			(at 1.27 12.49 0)
 			(layer "F.Fab")
 			(hide yes)
@@
 		)
 		(property "Value" "Conn_01x02"
-			(at 0 7.5 360)
+			(at 0 7.5 0)
 			(layer "F.Fab")
 			(hide yes)
@@
 		(locked yes)
 		(layer "F.Cu")
-		(at 159.1 117.615 180)
+		(at 159.38 117.615 180)
 		(descr "Through hole straight pin header, 1x02, 2.54mm pitch, single row")
 		(tags "Through hole pin header THT 1x02 2.54mm single row")
 		(property "Reference" "powerIN2"
-			(at -1 -3.46 360)
+			(at -1 -3.46 0)
 			(layer "F.SilkS")
 			(hide yes)
@@
 		)
 		(property "Value" "Conn_01x02"
-			(at 0 4.87 360)
+			(at 0 4.87 0)
 			(layer "F.Fab")
 			(hide yes)
@@
 		)
 		(property "Value" "Conn_02x05_Counter_Clockwise"
-			(at 1.27 12.49 360)
+			(at 1.27 12.49 0)
 			(layer "F.Fab")
 			(hide yes)
@@
 	)
 	(footprint "Module:Arduino_Nano"
+		(locked yes)
 		(layer "F.Cu")
 		(at 154.25 109.3 180)
@@
 	)
 	(gr_circle
-		(center 159.1 122.49)
-		(end 161.1 122.49)
+		(center 159.38 122.49)
+		(end 161.38 122.49)
 		(stroke
 			(width 0.05)
@@
 	)
 	(gr_rect
-		(start 129.6 66.14)
-		(end 163.5 131.915)
+		(start 129.14 65.9116)
+		(end 164.14 130.9116)
 		(stroke
 			(width 0.05)
@@
 	)
 	(gr_circle
-		(center 159.1 68.6775)
-		(end 161.1 68.6775)
+		(center 159.1 69.14)
+		(end 161.1 69.14)
 		(stroke
 			(width 0.05)
@@
 	)
 	(gr_circle
-		(center 133.9 68.6775)
-		(end 135.9 68.6775)
+		(center 133.9 69.14)
+		(end 135.9 69.14)
 		(stroke
 			(width 0.05)

Commit message: Updates
Routing:
- added copper zone on B.Cu, net (none)
- added copper zone on F.Cu, net (none)
Changed lines of the file:
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@@
 		(net 29)
 	)
+	(zone
+		(net 0)
+		(net_name "")
+		(layers "F&B.Cu")
+		(hatch edge 0.5)
+		(connect_pads
+			(clearance 0.5)
+		)
+		(min_thickness 0.25)
+		(filled_areas_thickness no)
+		(fill yes
+			(thermal_gap 0.5)
+			(thermal_bridge_width 0.5)
+			(island_removal_mode 1)
+			(island_area_min 10)
+		)
+		(polygon
+			(pts
+				(xy 109.78 57.14) (xy 181.28 58.64) (xy 176.28 139.64) (xy 105.78 133.14)
+			)
+		)
+	)
 )
