File: CAD/kiCAD/solarRadiationShield/solarRadiationShield.kicad_pcb (KiCad board)
At the start: 2 copper layers, 4 parts, among them J3 INSIG

Commit message: Big Updates
Parts:
- removed J3: INSIG, Connector_PinHeader_2.54mm:PinHeader_1x04_P2.54mm_Vertical
- added INSIG1: INSIG, Connector_PinHeader_2.54mm:PinHeader_1x04_P2.54mm_Vertical, F.Cu at (126.6, 77.8)
- moved lpsExtraFunc1 22.4 mm to (134.2, 91.9), turned to 180 degrees
- moved AHT20 22.1 mm to (133.4, 101.7)
- moved LPS331AP1 15.3 mm to (126.6, 102.1), turned to 180 degrees
Routing:
- net SDA: track 0.00 -> 42.5 mm, vias 0 -> 1
- net SCL: track 0.00 -> 40.3 mm, vias 0 -> 2
- net VDD: track 0.00 -> 38.6 mm
- net +3.3V: track 0.00 -> 36.8 mm, vias 0 -> 1
- net GND: track 0.00 -> 34.2 mm, vias 0 -> 3
- net SDO/SA0: track 0.00 -> 12.8 mm
- net INT1: track 0.00 -> 12.6 mm
- net INT2: track 0.00 -> 8.52 mm
- net CS: track 0.00 -> 8.52 mm
- added copper zone on B.Cu, net (none)
- added copper zone on F.Cu, net (none)
Other:
- board outline added: 13 x 37 mm

Commit message: updates
Other:
- outline, holes or cut-outs redrawn
Changed lines of the file:
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@@
 	(gr_circle
 		(center 127.05 108.475)
-		(end 129.15 108.475)
+		(end 129.05 108.475)
 		(stroke
 			(width 0.05)
