File: CAD/kiCAD/windVane/windVane.kicad_sch (KiCad schematic)
At the start: 10 parts

Commit message: Update Schematics
Parts:
- removed East1, NorthWest1, South1, SouthEast1, SouthWest1, West1: Conn_01x03, Connector_PinHeader_2.54mm:PinHeader_1x03_P2.54mm_Vertical, symbol Connector_Generic:Conn_01x03
- added C1, C2, C3, C4, C5, C6, C7, C8: 100nF, symbol Device:C
- added East, NorthWest, South, SouthEast, SouthWest, West: Conn_01x03, Connector_PinHeader_2.54mm:PinHeader_1x03_P2.54mm_Vertical, symbol Connector_Generic:Conn_01x03
- added R1, R2, R3, R4, R5, R6, R7, R8: 10k, symbol Device:R
Connections:
- net East: now also East.3 (Pin_3), R3.2
- net GND: now also C1.1, C2.1, C3.1, C4.1, C5.1, C6.1, C7.1, C8.1, East.2 (Pin_2), NorthWest.2 (Pin_2), South.2 (Pin_2), SouthEast.2 (Pin_2), SouthWest.2 (Pin_2), West.2 (Pin_2)
- net North: now also R1.2
- net NorthEast: now also R2.2
- net NorthWest: now also NorthWest.3 (Pin_3), R8.2
- net Q_{h}: now also SIG1.6 (Pin_6)
- net South: now also R5.2, South.3 (Pin_3)
- net SouthEast: now also R4.2, SouthEast.3 (Pin_3)
- net SouthWest: now also R6.2, SouthWest.3 (Pin_3)
- net Vdd: now also C1.2, C2.2, C3.2, C4.2, C5.2, C6.2, C7.2, C8.2, East.1 (Pin_1), NorthWest.1 (Pin_1), R1.1, R2.1, R3.1, R4.1, R5.1, R6.1, R7.1, R8.1, South.1 (Pin_1), SouthEast.1 (Pin_1), SouthWest.1 (Pin_1), West.1 (Pin_1)
- net West: now also R7.2, West.3 (Pin_3)
- net ~{Q}_{h}: no longer SIG1.6 (Pin_6)
Other:
- moved on the sheet: North1, SIG1, SN74HC165

Commit message: Updates
Parts:
- added J1, J2: Conn_01x01, Connector_PinHeader_2.54mm:PinHeader_1x01_P2.54mm_Vertical, symbol Connector_Generic:Conn_01x01
- C1, C2, C3, C4, C5, C6, C7, C8: footprint (none) -> Capacitor_SMD:C_0402_1005Metric
- R1, R2, R3, R4, R5, R6, R7, R8: footprint (none) -> Resistor_SMD:R_0402_1005Metric
- renumbered East to East1, NorthWest to NorthWest1, South to South1, SouthEast to SouthEast1, SouthWest to SouthWest1, West to West1
Connections:
- net SER: now also J2.1 (Pin_1)
- net ~{Q}_{h}: now also J1.1 (Pin_1)
Changed lines of the file:
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@@
+		)
+	)
+	(global_label "~{Q}_{h}"
+		(shape input)
+		(at 67.31 125.73 0)
+		(fields_autoplaced yes)
+		(effects
+			(font
+				(size 1.27 1.27)
+			)
+			(justify left)
+		)
+		(property "Intersheetrefs" "${INTERSHEET_REFS}"
+			(at 72.5957 125.73 0)
+			(effects
+				(font
+					(size 1.27 1.27)
+				)
+				(justify left)
+				(hide yes)
+			)
 		)
 	)
@@
 		)
 	)
+	(global_label "SER"
+		(shape input)
+		(at 67.31 138.43 0)
+		(fields_autoplaced yes)
+		(effects
+			(font
+				(size 1.27 1.27)
+			)
+			(justify left)
+		)
+		(property "Intersheetrefs" "${INTERSHEET_REFS}"
+			(at 73.9237 138.43 0)
+			(effects
+				(font
+					(size 1.27 1.27)
+				)
+				(justify left)
+				(hide yes)
+			)
+		)
+	)
 	(global_label "Vdd"
 		(shape input)
@@
 			)
 		)
-		(property "Footprint" ""
+		(property "Footprint" "Resistor_SMD:R_0402_1005Metric"
 			(at 164.338 63.5 90)
 			(effects
@@
 			)
 		)
-		(property "Footprint" ""
+		(property "Footprint" "Capacitor_SMD:C_0402_1005Metric"
 			(at 195.8848 91.44 0)
 			(effects
@@
 		(on_board yes)
 		(dnp no)
-		(property "Reference" "SouthEast"
+		(property "Reference" "SouthEast1"
 			(at 200.914 51.308 90)
 			(effects
@@
 			(project "windVane"
 				(path "/2de267c0-3460-4ea6-9140-c6cfbd374169"
-					(reference "SouthEast")
+					(reference "SouthEast1")
 					(unit 1)
 				)
@@
 			)
 		)
-		(property "Footprint" ""
+		(property "Footprint" "Resistor_SMD:R_0402_1005Metric"
 			(at 90.678 63.5 90)
 			(effects
@@
 			)
 		)
-		(property "Footprint" ""
+		(property "Footprint" "Capacitor_SMD:C_0402_1005Metric"
 			(at 84.1248 91.44 0)
 			(effects
@@
 			)
 		)
-		(property "Footprint" ""
+		(property "Footprint" "Resistor_SMD:R_0402_1005Metric"
 			(at 91.948 95.25 90)
 			(effects
@@
 			)
 		)
-		(property "Footprint" ""
+		(property "Footprint" "Resistor_SMD:R_0402_1005Metric"
 			(at 202.438 63.5 90)
 			(effects
@@
 			)
 		)
-		(property "Footprint" ""
+		(property "Footprint" "Resistor_SMD:R_0402_1005Metric"
 			(at 130.048 95.25 90)
 			(effects
@@
 			)
 		)
-		(property "Footprint" ""
-			(at 82.8548 59.69 0)
+		(property "Footprint" "Capacitor_SMD:C_0402_1005Metric"
+			(at 62.738 64.008 0)
 			(effects
 				(font
@@
 		(on_board yes)
 		(dnp no)
-		(property "Reference" "NorthWest"
+		(property "Reference" "NorthWest1"
 			(at 202.184 83.058 90)
 			(effects
@@
 			(project "windVane"
 				(path "/2de267c0-3460-4ea6-9140-c6cfbd374169"
-					(reference "NorthWest")
+					(reference "NorthWest1")
 					(unit 1)
 				)
@@
 		(on_board yes)
 		(dnp no)
-		(property "Reference" "South"
+		(property "Reference" "South1"
 			(at 90.424 83.058 90)
 			(effects
@@
 			(project "windVane"
 				(path "/2de267c0-3460-4ea6-9140-c6cfbd374169"
-					(reference "South")
+					(reference "South1")
+					(unit 1)
+				)
+			)
+		)
+	)
+	(symbol
+		(lib_id "Connector_Generic:Conn_01x01")
+		(at 62.23 138.43 0)
+		(mirror y)
+		(unit 1)
+		(exclude_from_sim no)
+		(in_bom yes)
+		(on_board yes)
+		(dnp no)
+		(fields_autoplaced yes)
+		(property "Reference" "J2"
+			(at 62.23 132.08 0)
+			(effects
+				(font
+					(size 1.27 1.27)
+				)
+			)
+		)
+		(property "Value" "Conn_01x01"
+			(at 62.23 134.62 0)
+			(effects
+				(font
+					(size 1.27 1.27)
+				)
+			)
+		)
+		(property "Footprint" "Connector_PinHeader_2.54mm:PinHeader_1x01_P2.54mm_Vertical"
+			(at 62.23 138.43 0)
+			(effects
+				(font
+					(size 1.27 1.27)
+				)
+				(hide yes)
+			)
+		)
+		(property "Datasheet" "~"
+			(at 62.23 138.43 0)
+			(effects
+				(font
+					(size 1.27 1.27)
+				)
+				(hide yes)
+			)
+		)
+		(property "Description" "Generic connector, single row, 01x01, script generated (kicad-library-utils/schlib/autogen/connector/)"
+			(at 62.23 138.43 0)
+			(effects
+				(font
+					(size 1.27 1.27)
+				)
+				(hide yes)
+			)
+		)
+		(pin "1"
+		)
+		(instances
+			(project "windVane"
+				(path "/2de267c0-3460-4ea6-9140-c6cfbd374169"
+					(reference "J2")
 					(unit 1)
 				)
@@
 			)
 		)
-		(property "Footprint" ""
+		(property "Footprint" "Resistor_SMD:R_0402_1005Metric"
 			(at 165.608 95.25 90)
 			(effects
@@
 			)
 		)
-		(property "Footprint" ""
+		(property "Footprint" "Capacitor_SMD:C_0402_1005Metric"
 			(at 194.6148 59.69 0)
 			(effects
@@
 		(on_board yes)
 		(dnp no)
-		(property "Reference" "East"
+		(property "Reference" "East1"
 			(at 162.814 51.308 90)
 			(effects
@@
 			(project "windVane"
 				(path "/2de267c0-3460-4ea6-9140-c6cfbd374169"
-					(reference "East")
+					(reference "East1")
 					(unit 1)
 				)
@@
 		(on_board yes)
 		(dnp no)
-		(property "Reference" "West"
+		(property "Reference" "West1"
 			(at 164.084 83.058 90)
 			(effects
@@
 			(project "windVane"
 				(path "/2de267c0-3460-4ea6-9140-c6cfbd374169"
-					(reference "West")
+					(reference "West1")
 					(unit 1)
 				)
@@
 			)
 		)
-		(property "Footprint" ""
+		(property "Footprint" "Resistor_SMD:R_0402_1005Metric"
 			(at 128.778 63.5 90)
 			(effects
@@
 			)
 		)
-		(property "Footprint" ""
+		(property "Footprint" "Resistor_SMD:R_0402_1005Metric"
 			(at 203.708 95.25 90)
 			(effects
@@
 	)
 	(symbol
+		(lib_id "Connector_Generic:Conn_01x01")
+		(at 62.23 125.73 0)
+		(mirror y)
+		(unit 1)
+		(exclude_from_sim no)
+		(in_bom yes)
+		(on_board yes)
+		(dnp no)
+		(fields_autoplaced yes)
+		(property "Reference" "J1"
+			(at 62.23 119.38 0)
+			(effects
+				(font
+					(size 1.27 1.27)
+				)
+			)
+		)
+		(property "Value" "Conn_01x01"
+			(at 62.23 121.92 0)
+			(effects
+				(font
+					(size 1.27 1.27)
+				)
+			)
+		)
+		(property "Footprint" "Connector_PinHeader_2.54mm:PinHeader_1x01_P2.54mm_Vertical"
+			(at 62.23 125.73 0)
+			(effects
+				(font
+					(size 1.27 1.27)
+				)
+				(hide yes)
+			)
+		)
+		(property "Datasheet" "~"
+			(at 62.23 125.73 0)
+			(effects
+				(font
+					(size 1.27 1.27)
+				)
+				(hide yes)
+			)
+		)
+		(property "Description" "Generic connector, single row, 01x01, script generated (kicad-library-utils/schlib/autogen/connector/)"
+			(at 62.23 125.73 0)
+			(effects
+				(font
+					(size 1.27 1.27)
+				)
+				(hide yes)
+			)
+		)
+		(pin "1"
+		)
+		(instances
+			(project ""
+				(path "/2de267c0-3460-4ea6-9140-c6cfbd374169"
+					(reference "J1")
+					(unit 1)
+				)
+			)
+		)
+	)
+	(symbol
 		(lib_id "Connector_Generic:Conn_01x03")
 		(at 125.73 86.36 90)
@@
 		(on_board yes)
 		(dnp no)
-		(property "Reference" "SouthWest"
+		(property "Reference" "SouthWest1"
 			(at 128.524 83.058 90)
 			(effects
@@
 			(project "windVane"
 				(path "/2de267c0-3460-4ea6-9140-c6cfbd374169"
-					(reference "SouthWest")
+					(reference "SouthWest1")
 					(unit 1)
 				)
@@
 			)
 		)
-		(property "Footprint" ""
+		(property "Footprint" "Capacitor_SMD:C_0402_1005Metric"
 			(at 156.5148 59.69 0)
 			(effects
@@
 			)
 		)
-		(property "Footprint" ""
+		(property "Footprint" "Capacitor_SMD:C_0402_1005Metric"
 			(at 157.7848 91.44 0)
 			(effects
@@
 			)
 		)
-		(property "Footprint" ""
+		(property "Footprint" "Capacitor_SMD:C_0402_1005Metric"
 			(at 122.2248 91.44 0)
 			(effects
@@
 			)
 		)
-		(property "Footprint" ""
+		(property "Footprint" "Capacitor_SMD:C_0402_1005Metric"
 			(at 120.9548 59.69 0)
 			(effects

Commit message: Update
Connections:
- net North: now also SN74HC165.3 (Pin_3); no longer SN74HC165.11 (Pin_11)
- net NorthEast: now also SN74HC165.14 (Pin_14); no longer SN74HC165.3 (Pin_3)
- net NorthWest: now also SN74HC165.4 (Pin_4); no longer SN74HC165.5 (Pin_5)
- net South: now also SN74HC165.11 (Pin_11); no longer SN74HC165.12 (Pin_12)
- net SouthEast: now also SN74HC165.12 (Pin_12); no longer SN74HC165.4 (Pin_4)
- net West: now also SN74HC165.5 (Pin_5); no longer SN74HC165.14 (Pin_14)
Changed lines of the file:
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@@
 	(global_label "West"
 		(shape input)
-		(at 118.11 123.19 0)
-		(fields_autoplaced yes)
-		(effects
-			(font
-				(size 1.27 1.27)
-			)
-			(justify left)
-		)
-		(property "Intersheetrefs" "${INTERSHEET_REFS}"
-			(at 125.389 123.19 0)
-			(effects
-				(font
-					(size 1.27 1.27)
-				)
-				(justify left)
+		(at 105.41 128.27 180)
+		(fields_autoplaced yes)
+		(effects
+			(font
+				(size 1.27 1.27)
+			)
+			(justify right)
+		)
+		(property "Intersheetrefs" "${INTERSHEET_REFS}"
+			(at 98.131 128.27 0)
+			(effects
+				(font
+					(size 1.27 1.27)
+				)
+				(justify right)
 				(hide yes)
 			)
@@
 	(global_label "South"
 		(shape input)
-		(at 118.11 128.27 0)
-		(fields_autoplaced yes)
-		(effects
-			(font
-				(size 1.27 1.27)
-			)
-			(justify left)
-		)
-		(property "Intersheetrefs" "${INTERSHEET_REFS}"
-			(at 126.4774 128.27 0)
+		(at 118.11 130.81 0)
+		(fields_autoplaced yes)
+		(effects
+			(font
+				(size 1.27 1.27)
+			)
+			(justify left)
+		)
+		(property "Intersheetrefs" "${INTERSHEET_REFS}"
+			(at 126.4774 130.81 0)
 			(effects
 				(font
@@
 	(global_label "North"
 		(shape input)
-		(at 118.11 130.81 0)
-		(fields_autoplaced yes)
-		(effects
-			(font
-				(size 1.27 1.27)
-			)
-			(justify left)
-		)
-		(property "Intersheetrefs" "${INTERSHEET_REFS}"
-			(at 126.2356 130.81 0)
-			(effects
-				(font
-					(size 1.27 1.27)
-				)
-				(justify left)
+		(at 105.41 123.19 180)
+		(fields_autoplaced yes)
+		(effects
+			(font
+				(size 1.27 1.27)
+			)
+			(justify right)
+		)
+		(property "Intersheetrefs" "${INTERSHEET_REFS}"
+			(at 97.2844 123.19 0)
+			(effects
+				(font
+					(size 1.27 1.27)
+				)
+				(justify right)
 				(hide yes)
 			)
@@
 	(global_label "NorthWest"
 		(shape input)
-		(at 105.41 128.27 180)
-		(fields_autoplaced yes)
-		(effects
-			(font
-				(size 1.27 1.27)
-			)
-			(justify right)
-		)
-		(property "Intersheetrefs" "${INTERSHEET_REFS}"
-			(at 92.9906 128.27 0)
+		(at 105.41 125.73 180)
+		(fields_autoplaced yes)
+		(effects
+			(font
+				(size 1.27 1.27)
+			)
+			(justify right)
+		)
+		(property "Intersheetrefs" "${INTERSHEET_REFS}"
+			(at 92.9906 125.73 0)
 			(effects
 				(font
@@
 	(global_label "NorthEast"
 		(shape input)
-		(at 105.41 123.19 180)
-		(fields_autoplaced yes)
-		(effects
-			(font
-				(size 1.27 1.27)
-			)
-			(justify right)
-		)
-		(property "Intersheetrefs" "${INTERSHEET_REFS}"
-			(at 93.2326 123.19 0)
-			(effects
-				(font
-					(size 1.27 1.27)
-				)
-				(justify right)
+		(at 118.11 123.19 0)
+		(fields_autoplaced yes)
+		(effects
+			(font
+				(size 1.27 1.27)
+			)
+			(justify left)
+		)
+		(property "Intersheetrefs" "${INTERSHEET_REFS}"
+			(at 130.2874 123.19 0)
+			(effects
+				(font
+					(size 1.27 1.27)
+				)
+				(justify left)
 				(hide yes)
 			)
@@
 	(global_label "SouthEast"
 		(shape input)
-		(at 105.41 125.73 180)
-		(fields_autoplaced yes)
-		(effects
-			(font
-				(size 1.27 1.27)
-			)
-			(justify right)
-		)
-		(property "Intersheetrefs" "${INTERSHEET_REFS}"
-			(at 92.9908 125.73 0)
-			(effects
-				(font
-					(size 1.27 1.27)
-				)
-				(justify right)
-				(hide yes)
-			)
+		(at 118.11 128.27 0)
+		(fields_autoplaced yes)
+		(effects
+			(font
+				(size 1.27 1.27)
+			)
+			(justify left)
+		)
+		(property "Intersheetrefs" "${INTERSHEET_REFS}"
+			(at 130.5292 128.27 0)
+			(effects
+				(font
+					(size 1.27 1.27)
+				)
+				(justify left)
+				(hide yes)
+			)
