File: CAD/kiCAD/windVane/windVane.kicad_pcb (KiCad board)
At the start: 2 copper layers, 10 parts

Commit message: Updates
Parts:
- added C1: 100nF, Capacitor_SMD:C_0402_1005Metric, F.Cu at (150.5, 82.5)
- added C2: 100nF, Capacitor_SMD:C_0402_1005Metric, F.Cu at (160.0, 91.0)
- added C3: 100nF, Capacitor_SMD:C_0402_1005Metric, F.Cu at (163.5, 100.8)
- added C4: 100nF, Capacitor_SMD:C_0402_1005Metric, F.Cu at (160.3, 111.2)
- added C5: 100nF, Capacitor_SMD:C_0402_1005Metric, F.Cu at (150.2, 114.5)
- added C6: 100nF, Capacitor_SMD:C_0402_1005Metric, F.Cu at (139.2, 110.2)
- added C7: 100nF, Capacitor_SMD:C_0402_1005Metric, F.Cu at (137.0, 101.0)
- added C8: 100nF, Capacitor_SMD:C_0402_1005Metric, F.Cu at (140.8, 89.7)
- added J1: Conn_01x01, Connector_PinHeader_2.54mm:PinHeader_1x01_P2.54mm_Vertical, F.Cu at (143.0, 104.4)
- added J2: Conn_01x01, Connector_PinHeader_2.54mm:PinHeader_1x01_P2.54mm_Vertical, F.Cu at (157.0, 104.4)
- added R1: 10k, Resistor_SMD:R_0402_1005Metric, F.Cu at (148.0, 82.5)
- added R2: 10k, Resistor_SMD:R_0402_1005Metric, F.Cu at (158.5, 89.0)
- added R3: 10k, Resistor_SMD:R_0402_1005Metric, F.Cu at (163.5, 103.0)
- added R4: 10k, Resistor_SMD:R_0402_1005Metric, F.Cu at (161.6, 109.9)
- added R5: 10k, Resistor_SMD:R_0402_1005Metric, F.Cu at (148.0, 114.5)
- added R6: 10k, Resistor_SMD:R_0402_1005Metric, F.Cu at (137.6, 108.6)
- added R7: 10k, Resistor_SMD:R_0402_1005Metric, F.Cu at (137.0, 99.0)
- added R8: 10k, Resistor_SMD:R_0402_1005Metric, F.Cu at (138.0, 92.5)
- SIG1: moved to B.Cu
- moved East1 64.4 mm to (166.0, 103.5), turned to 180 degrees
- moved SIG1 58.5 mm to (143.7, 111.0), turned to -90 degrees
- moved NorthEast1 49.8 mm to (163.8, 90.8), turned to -135 degrees
- moved SouthEast1 48.5 mm to (160.2, 114.8), turned to 135 degrees
- moved South1 46.6 mm to (147.5, 117.0), turned to 90 degrees
- moved SouthWest1 34.2 mm to (136.2, 111.2), turned to 45 degrees
- moved NorthWest1 29.8 mm to (139.8, 87.2), turned to -45 degrees
- moved SN74HC165 26.1 mm to (146.2, 89.1)
- moved West1 25.1 mm to (134.0, 98.5)
- moved North1 16.5 mm to (152.5, 85.0), turned to -90 degrees
Connections:
- NorthWest1 pad 3: NorhtWest -> NorthWest
- SIG1 pad 6: ~{Q}_{h} -> Q_{h}
Routing:
- net SH/~{LD}: track 0.00 -> 26.0 mm
- net clkINH: track 0.00 -> 23.0 mm
- net CLK: track 0.00 -> 22.2 mm
- net Q_{h}: track 0.00 -> 6.31 mm
- net GND: track 0.00 -> 4.10 mm
- net ~{Q}_{h}: track 0.00 -> 3.20 mm
- net SER: track 0.00 -> 3.18 mm
- net NorthWest: track 0.00 -> 2.66 mm
Other:
- board outline added: 40 x 40 mm
- board text added: "+3.3 V"
- board text added: "CLK"
- board text added: "CLKINH"
- board text added: "GND"
- board text added: "Q_{h}"
- board text added: "SH/~{LD}"

Commit message: Update
Parts:
- moved R5 6.40 mm to (152.0, 119.5)
- moved R6 5.42 mm to (141.2, 112.8), turned to -45 degrees
- moved C5 5.00 mm to (150.0, 119.5)
- moved R3 4.11 mm to (163.5, 98.9)
- moved R7 4.02 mm to (136.6, 103.0)
- moved C8 1.54 mm to (139.8, 90.8)
- moved C6 1.27 mm to (139.7, 111.3), turned to -45 degrees
- moved R8 0.55 mm to (138.4, 92.1)
- moved C1 0.52 mm to (150.0, 82.5), turned to 180 degrees
- moved C2 0.50 mm to (160.0, 90.5)
- moved C7 0.40 mm to (136.6, 101.0), turned to -90 degrees
- moved C3 0.13 mm to (163.5, 100.9)
Connections:
- SN74HC165 pad 11: North -> South
- SN74HC165 pad 12: South -> SouthEast
- SN74HC165 pad 14: West -> NorthEast
- SN74HC165 pad 3: NorthEast -> North
- SN74HC165 pad 4: SouthEast -> NorthWest
- SN74HC165 pad 5: NorthWest -> West
Routing:
- net GND: track 4.10 -> 176.6 mm
- net Vdd: track 0.00 -> 149.5 mm
- net SouthWest: track 0.00 -> 24.1 mm
- net SouthEast: track 0.00 -> 21.3 mm
- net South: track 0.00 -> 20.9 mm
- net West: track 0.00 -> 17.0 mm
- net East: track 0.00 -> 15.4 mm
- net North: track 0.00 -> 13.4 mm
- net NorthEast: track 0.00 -> 13.0 mm
- net NorthWest: track 2.66 -> 15.2 mm
- added copper zone on B.Cu, net (none)
- added copper zone on F.Cu, net (none)

Commit message: updates
Parts:
- moved J1 1.64 mm to (143.0, 106.0)
- moved J2 1.64 mm to (157.0, 106.0)
Routing:
- net West: track 17.0 -> 19.9 mm
- net ~{Q}_{h}: track 3.20 -> 4.54 mm
- net SER: track 3.18 -> 4.52 mm
Other:
- outline, holes or cut-outs redrawn
Changed lines of the file:
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@@
 		(tags "capacitor")
 		(property "Reference" "C1"
-			(at 0 -1.16 360)
+			(at 0 -1.16 0)
 			(layer "F.SilkS")
 			(hide yes)
@@
 		)
 		(property "Value" "100nF"
-			(at 0 1.16 360)
+			(at 0 1.16 0)
 			(layer "F.Fab")
 			(effects
@@
 		)
 		(fp_text user "${REFERENCE}"
-			(at 0 0 360)
+			(at 0 0 0)
 			(layer "F.Fab")
 			(effects
@@
 		(tags "resistor")
 		(property "Reference" "R5"
-			(at 0 -1.17 360)
+			(at 0 -1.17 0)
 			(layer "F.SilkS")
 			(hide yes)
@@
 		)
 		(property "Value" "10k"
-			(at 0 1.17 360)
+			(at 0 1.17 0)
 			(layer "F.Fab")
 			(effects
@@
 		)
 		(fp_text user "${REFERENCE}"
-			(at 0 0 360)
+			(at 0 0 0)
 			(layer "F.Fab")
 			(effects
@@
 	(footprint "Connector_PinHeader_2.54mm:PinHeader_1x01_P2.54mm_Vertical"
 		(layer "F.Cu")
-		(at 143 104.365)
+		(at 143 106)
 		(descr "Through hole straight pin header, 1x01, 2.54mm pitch, single row")
 		(tags "Through hole pin header THT 1x01 2.54mm single row")
@@
 		(tags "capacitor")
 		(property "Reference" "C5"
-			(at 0 -1.16 360)
+			(at 0 -1.16 0)
 			(layer "F.SilkS")
 			(hide yes)
@@
 		)
 		(property "Value" "100nF"
-			(at 0 1.16 360)
+			(at 0 1.16 0)
 			(layer "F.Fab")
 			(effects
@@
 		)
 		(fp_text user "${REFERENCE}"
-			(at 0 0 360)
+			(at 0 0 0)
 			(layer "F.Fab")
 			(effects
@@
 	(footprint "Connector_PinHeader_2.54mm:PinHeader_1x01_P2.54mm_Vertical"
 		(layer "F.Cu")
-		(at 157 104.365)
+		(at 157 106)
 		(descr "Through hole straight pin header, 1x01, 2.54mm pitch, single row")
 		(tags "Through hole pin header THT 1x01 2.54mm single row")
@@
 	)
 	(gr_rect
-		(start 138 89)
-		(end 162 113)
+		(start 157 99)
+		(end 161 103)
 		(stroke
-			(width 0.1)
+			(width 0.05)
 			(type default)
 		)
 		(fill none)
-		(layer "Dwgs.User")
+		(layer "Edge.Cuts")
 	)
 	(gr_circle
@@
 		(layer "Edge.Cuts")
 	)
+	(gr_rect
+		(start 139 99)
+		(end 143 103)
+		(stroke
+			(width 0.05)
+			(type default)
+		)
+		(fill none)
+		(layer "Edge.Cuts")
+	)
 	(gr_text "+3.3 V"
 		(at 143.5 112.5 135)
@@
 	)
 	(segment
-		(start 159 106.407898)
-		(end 159 99.8)
+		(start 153.82 99.285)
+		(end 155.485 99.285)
 		(width 0.2)
 		(layer "B.Cu")
@@
 	)
 	(segment
-		(start 159 99.8)
-		(end 158.485 99.285)
+		(start 155.6 103.4)
+		(end 155.6 99.4)
 		(width 0.2)
 		(layer "B.Cu")
@@
 	)
 	(segment
-		(start 158.485 99.285)
-		(end 153.82 99.285)
+		(start 158 104)
+		(end 156.2 104)
+		(width 0.2)
+		(layer "B.Cu")
+		(net 7)
+	)
+	(segment
+		(start 159 104.4)
+		(end 158.6 104)
+		(width 0.2)
+		(layer "B.Cu")
+		(net 7)
+	)
+	(segment
+		(start 159 106.407898)
+		(end 159 104.4)
+		(width 0.2)
+		(layer "B.Cu")
+		(net 7)
+	)
+	(segment
+		(start 155.485 99.285)
+		(end 155.6 99.4)
+		(width 0.2)
+		(layer "B.Cu")
+		(net 7)
+	)
+	(segment
+		(start 158.6 104)
+		(end 158 104)
+		(width 0.2)
+		(layer "B.Cu")
+		(net 7)
+	)
+	(segment
+		(start 156.2 104)
+		(end 155.6 103.4)
 		(width 0.2)
 		(layer "B.Cu")
@@
 	)
 	(segment
-		(start 146.2 99.285)
-		(end 142.315 99.285)
+		(start 143.8 104)
+		(end 134.445 104)
 		(width 0.2)
 		(layer "B.Cu")
@@
 	)
 	(segment
-		(start 142.315 99.285)
-		(end 138.045 103.555)
+		(start 134.445 104)
+		(end 134 103.555)
 		(width 0.2)
 		(layer "B.Cu")
@@
 	)
 	(segment
-		(start 138.045 103.555)
-		(end 134 103.555)
+		(start 144.215 99.285)
+		(end 144 99.5)
+		(width 0.2)
+		(layer "B.Cu")
+		(net 9)
+	)
+	(segment
+		(start 144 99.5)
+		(end 144 103.8)
+		(width 0.2)
+		(layer "B.Cu")
+		(net 9)
+	)
+	(segment
+		(start 146.2 99.285)
+		(end 144.215 99.285)
+		(width 0.2)
+		(layer "B.Cu")
+		(net 9)
+	)
+	(segment
+		(start 144 103.8)
+		(end 143.8 104)
 		(width 0.2)
 		(layer "B.Cu")
@@
 	(segment
 		(start 146.2 104.365)
-		(end 143 104.365)
+		(end 143.5 104.365)
+		(width 0.2)
+		(layer "F.Cu")
+		(net 11)
+	)
+	(segment
+		(start 143 104.865)
+		(end 143.5 104.365)
+		(width 0.2)
+		(layer "F.Cu")
+		(net 11)
+	)
+	(segment
+		(start 143 106)
+		(end 143 104.865)
 		(width 0.2)
 		(layer "F.Cu")
@@
 	(segment
 		(start 153.82 104.365)
-		(end 157 104.365)
+		(end 156.5 104.365)
+		(width 0.2)
+		(layer "F.Cu")
+		(net 13)
+	)
+	(segment
+		(start 157 106)
+		(end 157 104.865)
+		(width 0.2)
+		(layer "F.Cu")
+		(net 13)
+	)
+	(segment
+		(start 157 104.865)
+		(end 156.5 104.365)
 		(width 0.2)
 		(layer "F.Cu")
