File: CAD/kiCAD/powerSystem/powerSystem.kicad_pcb (KiCad board)
At the start: 2 copper layers, 39 x 17 mm, 11 parts, among them P1 Conn_01x02, P2 Conn_01x02, P3 Conn_01x02, P4 Conn_01x02

Commit message: Updates
Routing:
- added copper zone on B.Cu, net (none)
- added copper zone on F.Cu, net (none)
Changed lines of the file:
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@@
 		(net 5)
 	)
+	(zone
+		(net 0)
+		(net_name "")
+		(layers "F&B.Cu")
+		(hatch edge 0.5)
+		(connect_pads
+			(clearance 0.5)
+		)
+		(min_thickness 0.25)
+		(filled_areas_thickness no)
+		(fill yes
+			(thermal_gap 0.5)
+			(thermal_bridge_width 0.5)
+			(island_removal_mode 1)
+			(island_area_min 10)
+		)
+		(polygon
+			(pts
+				(xy 138.2 80.2) (xy 187.2 80.2) (xy 189.2 116.2) (xy 138.2 113.2)
+			)
+		)
+	)
 )

Commit message: updates
Parts:
- moved SDO2 13.0 mm to (178.2, 88.6)
- moved SDI2 9.07 mm to (173.7, 88.6)
- moved P1 7.58 mm to (146.7, 96.8)
- moved P2 7.58 mm to (151.2, 96.8)
- moved P3 5.77 mm to (155.7, 96.8)
- moved P4 5.77 mm to (160.2, 96.8)
- moved SIGOUT1 4.93 mm to (164.7, 99.1)
- moved PMI1 4.42 mm to (164.7, 88.6)
- moved PMO1 4.42 mm to (169.2, 88.6)
- moved SDI1 4.42 mm to (155.7, 88.6)
- moved SDO1 4.42 mm to (160.2, 88.6)
Routing:
- net /GND: track 65.1 -> 48.6 mm
- net /+3_3V: track 5.88 -> 17.4 mm
- net /+5V: track 27.2 -> 18.1 mm
- net /0~10V: track 24.6 -> 23.7 mm
Other:
- board size 39 x 17 mm -> 43 x 20 mm
